Commit message: first attempt at lidar

File: model/robot.xacro (robot description, xacro)
@@ -27,4 +27,14 @@
     <xacro:property name="caster_inertia_y" value="${2.0/5.0 * caster_mass * caster_radius * caster_radius}"/>
     <xacro:property name="caster_inertia_z" value="${2.0/5.0 * caster_mass * caster_radius * caster_radius}"/>
+    <!-- Macros -->
+    <xacro:macro name="inertial_cylinder" params="mass length radius *origin">
+        <inertial>
+            <xacro:insert_block name="origin"/>
+            <mass value="${mass}" />
+            <inertia ixx="${(1/12) * mass * (3*radius*radius + length*length)}" ixy="0.0" ixz="0.0"
+                    iyy="${(1/12) * mass * (3*radius*radius + length*length)}" iyz="0.0"
+                    izz="${(1/2) * mass * (radius*radius)}" />
+        </inertial>
+    </xacro:macro>
     <!-- Control Parameters -->
     <xacro:property name="max_linear_acceleration" value="10"/>
@@ -142,4 +152,60 @@
     </joint>
     <!-- Laser -->
+     <joint name="laser_joint" type="fixed">
+        <parent link="body_link"/>
+        <child link="laser_frame"/>
+        <origin xyz="0.122 0 0.15" rpy="0 0 0"/>
+    </joint>
+    <link name="laser_frame">
+        <visual>
+            <geometry>
+                <cylinder radius="0.05" length="0.04"/>
+            </geometry>
+            <material name="black"/>
+        </visual>
+        <visual>
+            <origin xyz="0 0 -0.05"/>
+            <geometry>
+                <cylinder radius="0.01" length="0.1"/>
+            </geometry>
+            <material name="black"/>
+        </visual>
+        <collision>
+            <geometry>
+                <cylinder radius="0.05" length="0.04"/>
+            </geometry>
+        </collision>
+        <xacro:inertial_cylinder mass="0.1" length="0.04" radius="0.05">
+            <origin xyz="0 0 0" rpy="0 0 0"/>
+        </xacro:inertial_cylinder>
+    </link>
+    <gazebo reference="laser_frame">
+        <material>Gazebo/Black</material>
+        <sensor name="laser" type="ray">
+            <pose> 0 0 0 0 0 0 </pose>
+            <visualize>true</visualize>
+            <update_rate>10</update_rate>
+            <ray>
+                <scan>
+                    <horizontal>
+                        <samples>360</samples>
+                        <min_angle>-3.14</min_angle>
+                        <max_angle>3.14</max_angle>
+                    </horizontal>
+                </scan>
+                <range>
+                    <min>0.3</min>
+                    <max>12</max>
+                </range>
+            </ray>
+            <plugin name="laser_controller" filename="libgazebo_ros_ray_sensor.so">
+                <ros>
+                    <argument>~/out:=scan</argument>
+                </ros>
+                <output_type>sensor_msgs/LaserScan</output_type>
+                <frame_name>laser_frame</frame_name>
+            </plugin>
+        </sensor>
+    </gazebo>
     <!-- Caster Wheel Joint (fixed) -->
     <joint name="caster_joint" type="fixed">

Commit message: working lidar but no rviz visibility

File: model/robot.xacro (robot description, xacro)
@@ -181,30 +181,38 @@
     </link>
     <gazebo reference="laser_frame">
-        <material>Gazebo/Black</material>
-        <sensor name="laser" type="ray">
-            <pose> 0 0 0 0 0 0 </pose>
-            <visualize>true</visualize>
-            <update_rate>10</update_rate>
-            <ray>
-                <scan>
-                    <horizontal>
-                        <samples>360</samples>
-                        <min_angle>-3.14</min_angle>
-                        <max_angle>3.14</max_angle>
-                    </horizontal>
-                </scan>
-                <range>
-                    <min>0.3</min>
-                    <max>12</max>
-                </range>
-            </ray>
-            <plugin name="laser_controller" filename="libgazebo_ros_ray_sensor.so">
-                <ros>
-                    <argument>~/out:=scan</argument>
-                </ros>
-                <output_type>sensor_msgs/LaserScan</output_type>
-                <frame_name>laser_frame</frame_name>
-            </plugin>
-        </sensor>
+	  <selfCollide>false</selfCollide>
+      <mu1 value="0.05" />
+      <mu2 value="0.05" />
+    </gazebo>
+    <gazebo reference="laser_frame" >
+    <sensor name='gpu_lidar' type='gpu_lidar'>"
+        <pose relative_to='laser_frame'>0 0 0 0 0 0</pose>
+        <topic>scan</topic>
+        <update_rate>10</update_rate>
+        <lidar>
+            <scan>
+                <horizontal>
+                    <samples>640</samples>
+                    <resolution>1</resolution>
+                    <min_angle>-3.14</min_angle>
+                    <max_angle>3.14</max_angle>
+                </horizontal>
+                <vertical>
+                    <samples>1</samples>
+                    <resolution>0.01</resolution>
+                    <min_angle>0</min_angle>
+                    <max_angle>0</max_angle>
+                </vertical>
+            </scan>
+            <range>
+                <min>0.08</min>
+                <max>30.0</max>
+                <resolution>0.01</resolution>
+            </range>
+            <frame_id>/laser_frame</frame_id>
+        </lidar>
+        <always_on>1</always_on>
+        <visualize>true</visualize>
+    </sensor>
     </gazebo>
     <!-- Caster Wheel Joint (fixed) -->
@@ -243,4 +251,7 @@
             <odom_topic>odom</odom_topic>
         </plugin>
+        <plugin filename="gz-sim-sensors-system" name="gz::sim::systems::Sensors">
+            <render_engine>ogre2</render_engine>
+        </plugin>
         <plugin filename="gz-sim-joint-state-publisher-system" name="gz::sim::systems::JointStatePublisher">
             <topic>joint_states</topic>

Commit message: working mapping in rviz

File: model/robot.xacro (robot description, xacro)
@@ -40,6 +40,14 @@
     <xacro:property name="max_linear_acceleration" value="10"/>
     <!-- Links -->
-    <!-- Body Link -->
-    <link name="body_link">
+    <!-- BASE_FOOTPRINT LINK -->
+    <joint name="base_footprint_joint" type="fixed">
+        <parent link="base_link"/>
+        <child link="base_footprint"/>
+        <origin xyz="0 0 0" rpy="0 0 0"/>
+    </joint>
+    <link name="base_footprint">
+    </link>
+    <!-- Base Link -->
+    <link name="base_link">
         <visual>
             <origin xyz="0.0 0.0 0.0" rpy="0.0 0.0 0.0"/>
@@ -136,5 +144,5 @@
     <joint name="left_wheel_joint" type="continuous">
         <origin xyz="-${wheel_offset} ${wheel_separation/2} -${wheel_radius/2}" rpy="0 0 0"/>
-        <parent link="body_link"/>
+        <parent link="base_link"/>
         <child link="left_wheel_link"/>
         <axis xyz="0 1 0"/>
@@ -145,5 +153,5 @@
     <joint name="right_wheel_joint" type="continuous">
         <origin xyz="-${wheel_offset} ${-wheel_separation/2} -${wheel_radius/2}" rpy="0 0 0"/>
-        <parent link="body_link"/>
+        <parent link="base_link"/>
         <child link="right_wheel_link"/>
         <axis xyz="0 1 0"/>
@@ -153,5 +161,5 @@
     <!-- Laser -->
      <joint name="laser_joint" type="fixed">
-        <parent link="body_link"/>
+        <parent link="base_link"/>
         <child link="laser_frame"/>
         <origin xyz="0.122 0 0.15" rpy="0 0 0"/>
@@ -220,9 +228,9 @@
     <joint name="caster_joint" type="fixed">
         <origin xyz="${caster_offset} 0 -${caster_radius/2}" rpy="0 0 0"/>
-        <parent link="body_link"/>
+        <parent link="base_link"/>
         <child link="caster_link"/>
     </joint>
     <!-- Gazebo Parameters -->
-    <gazebo reference="body_link">
+    <gazebo reference="base_link">
         <mu1>1.0</mu1>
         <mu2>1.0</mu2>
@@ -251,5 +259,5 @@
             <topic>cmd_vel</topic>
             <frame_id>odom</frame_id>
-            <child_frame_id>body_link</child_frame_id>
+            <child_frame_id>base_link</child_frame_id>
             <odom_topic>odom</odom_topic>
             <tf_topic>/tf</tf_topic>

Commit message: removed old controller

File: model/robot.xacro (robot description, xacro)
@@ -248,19 +248,27 @@
         <mu2>0.000001</mu2>
     </gazebo>
+    <ros2_control name="GazeboSystem" type="system">
+            <hardware>
+                <plugin>gz_ros2_control/GazeboSimSystem</plugin>
+            </hardware>
+            <joint name="left_wheel_joint">
+                <command_interface name="velocity">
+                    <param name="min">-10</param>
+                    <param name="max">10</param>
+                </command_interface>
+                <state_interface name="velocity"/>
+                <state_interface name="position"/>
+            </joint>
+            <joint name="right_wheel_joint">
+                <command_interface name="velocity">
+                    <param name="min">-10</param>
+                    <param name="max">10</param>
+                </command_interface>
+                <state_interface name="velocity"/>
+                <state_interface name="position"/>
+            </joint>
+        </ros2_control>
     <!-- Gazebo Plugins -->
     <gazebo>
-        <plugin filename="gz-sim-diff-drive-system" name="gz::sim::systems::DiffDrive">
-            <right_joint>right_wheel_joint</right_joint>
-            <left_joint>left_wheel_joint</left_joint>
-            <wheel_separation>${wheel_separation}</wheel_separation>
-            <wheel_radius>${wheel_radius}</wheel_radius>
-            <max_linear_acceleration>${max_linear_acceleration}</max_linear_acceleration>
-            <odom_publish_frequency>30</odom_publish_frequency>
-            <topic>cmd_vel</topic>
-            <frame_id>odom</frame_id>
-            <child_frame_id>base_link</child_frame_id>
-            <odom_topic>odom</odom_topic>
-            <tf_topic>/tf</tf_topic>
-        </plugin>
         <plugin filename="gz-sim-sensors-system" name="gz::sim::systems::Sensors">
             <render_engine>ogre2</render_engine>
@@ -271,4 +279,8 @@
             <joint_name>left_wheel_joint</joint_name>
         </plugin>
+        <plugin name="gz_ros2_control::GazeboSimROS2ControlPlugin" filename="libgz_ros2_control-system.so">
+            <parameters>$(find differential_drive_robot)/config/my_controllers.yaml</parameters>
+            <parameters>$(find differential_drive_robot)/config/gaz_ros2_ctl_use_sim.yaml</parameters>
+        </plugin>
     </gazebo>
 </robot>

Commit message: working ros2_control

File: model/robot.xacro (robot description, xacro)
@@ -248,4 +248,32 @@
         <mu2>0.000001</mu2>
     </gazebo>
+    <ros2_control name="RealRobot" type="system">
+            <hardware>
+                <plugin>diffdrive_arduino/DiffDriveArduino</plugin>
+                <param name="left_wheel_name">left_wheel_joint</param>
+                <param name="right_wheel_name">right_wheel_joint</param>
+                <param name="loop_rate">30</param>
+                <param name="device">/dev/ttyACM0</param>
+                <param name="baud_rate">57600</param>
+                <param name="timeout_ms">1000</param>
+                <param name="enc_counts_per_rev">3436</param>
+            </hardware>
+            <joint name="left_wheel_joint">
+                <command_interface name="velocity">
+                    <param name="min">-10</param>
+                    <param name="max">10</param>
+                </command_interface>
+                <state_interface name="position"/>
+                <state_interface name="velocity"/>
+            </joint>
+            <joint name="right_wheel_joint">
+                <command_interface name="velocity">
+                    <param name="min">-10</param>
+                    <param name="max">10</param>
+                </command_interface>
+                <state_interface name="position"/>
+                <state_interface name="velocity"/>
+            </joint>
+    </ros2_control>
     <ros2_control name="GazeboSystem" type="system">
             <hardware>

Commit message: working diffdrive controller

File: model/robot.xacro (robot description, xacro)
@@ -256,5 +256,5 @@
                 <param name="device">/dev/ttyACM0</param>
                 <param name="baud_rate">57600</param>
-                <param name="timeout_ms">1000</param>
+                <param name="timeout">1000</param>
                 <param name="enc_counts_per_rev">3436</param>
             </hardware>
@@ -276,25 +276,4 @@
             </joint>
     </ros2_control>
-    <ros2_control name="GazeboSystem" type="system">
-            <hardware>
-                <plugin>gz_ros2_control/GazeboSimSystem</plugin>
-            </hardware>
-            <joint name="left_wheel_joint">
-                <command_interface name="velocity">
-                    <param name="min">-10</param>
-                    <param name="max">10</param>
-                </command_interface>
-                <state_interface name="velocity"/>
-                <state_interface name="position"/>
-            </joint>
-            <joint name="right_wheel_joint">
-                <command_interface name="velocity">
-                    <param name="min">-10</param>
-                    <param name="max">10</param>
-                </command_interface>
-                <state_interface name="velocity"/>
-                <state_interface name="position"/>
-            </joint>
-        </ros2_control>
     <!-- Gazebo Plugins -->
     <gazebo>
